File: hardware/LED_panel/panel_0/panel_0.kicad_pcb (KiCad board)
At the start: 2 copper layers, 115 x 75 mm, 44 parts, among them J0 Conn_01x02_Pin, J1 Conn_01x02_Pin, J2-1 Conn_01x02_Pin, J2-2 Conn_01x02_Pin

Commit message: add spi temp board and connector
Parts:
- added C1: 0.1uF, Capacitor_SMD:C_0805_2012Metric, F.Cu at (193.5, 109.8)
- added IC1: TMP126NDCKR, KiCad:SOT65P210X110-6N, F.Cu at (190.6, 112.4)
- added J2: Conn_01x08_Pin, Connector_Molex:Molex_PicoBlade_53261-0871_1x08-1MP_P1.25mm_Horizontal, F.Cu at (200.8, 108.5)
Routing:
- net Net-(IC1-SIO): track 0.00 -> 16.4 mm
- net Net-(IC1-GND): track 0.00 -> 14.1 mm
- net Net-(IC1-~{CS}): track 0.00 -> 11.2 mm
- net Net-(IC1-VDD): track 0.00 -> 10.3 mm
- net Net-(IC1-~{ALERT}): track 0.00 -> 7.68 mm
- net Net-(IC1-SCLK): track 0.00 -> 7.36 mm
- net Net-(J2-Pin_5): track 0.00 -> 4.67 mm

Commit message: added extra mounting points
Parts:
- added H10: MountingHole, MountingHole:MountingHole_2.2mm_M2, F.Cu at (150.0, 145.0)
- added H11: MountingHole, MountingHole:MountingHole_2.2mm_M2, F.Cu at (110.0, 145.0)
- added H5: MountingHole, MountingHole:MountingHole_3.2mm_M3, F.Cu at (165.8, 92.5)
- added H6: MountingHole, MountingHole:MountingHole_3.2mm_M3, F.Cu at (165.8, 157.5)
- added H7: MountingHole, MountingHole:MountingHole_2.2mm_M2, F.Cu at (129.9, 125.0)
- added H8: MountingHole, MountingHole:MountingHole_2.2mm_M2, F.Cu at (110.0, 105.0)
- added H9: MountingHole, MountingHole:MountingHole_2.2mm_M2, F.Cu at (150.0, 105.0)
