File: hardware/control/control.kicad_pcb (KiCad board)
At the start: 2 copper layers, 200 x 70 mm, 46 parts, among them IC1 TMUX4053DYYR, J0 43045-0412, J1 Conn_01x02_Pin, J11 Conn_01x04_Pin, J12 Camera Isolated triggers (ope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, J2 Conn_01x02_Pin, J3 Conn_01x02_Pin, J4 Conn_01x02_Pin, J5 Conn_01x05_Pin, J6 Conn_01x04_Pin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

Commit message: cleaning traces
Routing:
- net Net-(IC1-S1B): track 30.6 -> 33.9 mm
Changed lines of the file:
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@@
 	)
 	(segment
-		(start 190.648745 87.659592)
-		(end 189.823745 88.484592)
-		(width 0.2)
-		(layer "F.Cu")
-		(net "Net-(IC1-S1B)")
-	)
-	(segment
 		(start 206.998745 75.359592)
 		(end 205.336745 75.359592)
@@
 	)
 	(segment
-		(start 189.823745 88.484592)
+		(start 189.004592 89.504592)
 		(end 189.823745 89.504592)
 		(width 0.2)
@@
 	)
 	(segment
+		(start 188.340408 87.659592)
+		(end 188 88)
+		(width 0.2)
+		(layer "F.Cu")
+		(net "Net-(IC1-S1B)")
+	)
+	(segment
+		(start 188 88.5)
+		(end 189.004592 89.504592)
+		(width 0.2)
+		(layer "F.Cu")
+		(net "Net-(IC1-S1B)")
+	)
+	(segment
+		(start 190.648745 87.659592)
+		(end 188.340408 87.659592)
+		(width 0.2)
+		(layer "F.Cu")
+		(net "Net-(IC1-S1B)")
+	)
+	(segment
 		(start 190.648745 86.934592)
 		(end 190.648745 87.659592)
@@
 		(net "Net-(IC1-S1B)")
 	)
+	(segment
+		(start 188 88)
+		(end 188 88.5)
+		(width 0.2)
+		(layer "F.Cu")
+		(net "Net-(IC1-S1B)")
+	)
 	(via
 		(at 190.648745 87.659592)
@@
 	)
 	(segment
-		(start 112.915 56.49)
+		(start 113.1675 57.955)
 		(end 114.38 57.955)
 		(width 1.3)
@@
 	)
 	(segment
+		(start 114.38 57.955)
+		(end 117.38 57.955)
+		(width 1.3)
+		(layer "F.Cu")
+		(net "Net-(F1-Pad1)")
+	)
+	(segment
 		(start 100.04 56.49)
-		(end 112.915 56.49)
+		(end 111.7025 56.49)
 		(width 1.3)
 		(layer "F.Cu")
@@
 	)
 	(segment
-		(start 114.38 57.955)
-		(end 117.38 57.955)
+		(start 111.7025 56.49)
+		(end 113.1675 57.955)
 		(width 1.3)
 		(layer "F.Cu")
@@
 	)
 	(zone
+		(net "Net-(A1-D9)")
+		(layer "F.Cu")
+		(hatch none 0.1)
+		(priority 30000)
+		(attr
+			(teardrop
+				(type padvia)
+			)
+		)
+		(connect_pads yes
+			(clearance 0)
+		)
+		(min_thickness 0.0254)
+		(fill yes
+			(island_removal_mode 1)
+		)
+		(polygon
+			(pts
+				(xy 228.824893 71.199592) (xy 228.681089 71.194703) (xy 228.559584 71.180483) (xy 228.463436 71.159509)
+				(xy 228.380237 71.131602) (xy 228.238221 71.055517) (xy 228.067787 70.919674) (xy 227.877522 70.765067)
+				(xy 227.755096 70.68104) (xy 227.605862 70.594055) (xy 227.223893 71.299592) (xy 227.605862 72.005129)
+				(xy 227.841508 71.860162) (xy 228.067787 71.67951) (xy 228.206647 71.565952) (xy 228.278201 71.518212)
+				(xy 228.356759 71.477488) (xy 228.446516 71.444522) (xy 228.551662 71.420056) (xy 228.67639 71.404832)
+				(xy 228.824893 71.399592)
+			)
+		)
+	)
+	(zone
 		(net "Net-(IC1-D2)")
 		(layer "F.Cu")
@@
 	)
 	(zone
-		(net "Net-(IC1-S1B)")
-		(layer "F.Cu")
-		(hatch none 0.1)
-		(priority 30120)
-		(attr
-			(teardrop
-				(type padvia)
-			)
-		)
-		(connect_pads yes
-			(clearance 0)
-		)
-		(min_thickness 0.0254)
-		(fill yes
-			(island_removal_mode 1)
-		)
-		(polygon
-			(pts
-				(xy 189.723745 89.204592) (xy 189.725351 89.23064) (xy 189.724314 89.310805) (xy 189.708528 89.342045)
-				(xy 189.673745 89.354592) (xy 189.823745 89.505592) (xy 189.973745 89.354592) (xy 189.950403 89.349928)
-				(xy 189.934723 89.337281) (xy 189.920437 89.292378) (xy 189.922139 89.23064) (xy 189.923745 89.204592)
-			)
-		)
-	)
-	(zone
 		(net "Net-(J5-Pin_4)")
 		(layer "F.Cu")
@@
 	)
 	(zone
-		(net "Net-(A1-D9)")
-		(layer "F.Cu")
-		(hatch none 0.1)
-		(priority 30087)
-		(attr
-			(teardrop
-				(type padvia)
-			)
-		)
-		(connect_pads yes
-			(clearance 0)
-		)
-		(min_thickness 0.0254)
-		(fill yes
-			(island_removal_mode 1)
-		)
-		(polygon
-			(pts
-				(xy 231.117822 71.399592) (xy 231.314964 71.404241) (xy 231.475267 71.416781) (xy 231.741074 71.460549)
-				(xy 231.805783 71.474592) (xy 232.084121 71.526154) (xy 232.264317 71.543147) (xy 232.493745 71.549592)
-				(xy 232.718822 71.299592) (xy 231.752125 71.049592) (xy 231.769859 71.106418) (xy 231.772776 71.151204)
-				(xy 231.764905 71.180123) (xy 231.748516 71.202306) (xy 231.692183 71.229554) (xy 231.583549 71.237597)
-				(xy 231.385458 71.22021) (xy 231.117822 71.199592)
-			)
-		)
-	)
-	(zone
 		(net "Net-(IC1-D2)")
 		(layer "F.Cu")
@@
 	)
 	(zone
-		(net "Net-(IC1-S1B)")
-		(layer "F.Cu")
-		(hatch none 0.1)
-		(priority 30100)
-		(attr
-			(teardrop
-				(type padvia)
-			)
-		)
-		(connect_pads yes
-			(clearance 0)
-		)
-		(min_thickness 0.0254)
-		(fill yes
-			(island_removal_mode 1)
-		)
-		(polygon
-			(pts
-				(xy 190.297007 88.152751) (xy 190.36878 88.087791) (xy 190.429479 88.046502) (xy 190.533257 88.00691)
-				(xy 190.568643 87.998199) (xy 190.653647 87.975944) (xy 190.76355 87.936756) (xy 190.651267 87.65707)
-				(xy 190.371581 87.544787) (xy 190.316629 87.712982) (xy 190.310137 87.739695) (xy 190.293101 87.804773)
-				(xy 190.268561 87.866256) (xy 190.226171 87.932367) (xy 190.155586 88.01133)
-			)
-		)
-	)
-	(zone
 		(net "Net-(J4-Pin_1)")
 		(layer "F.Cu")
@@
 	)
 	(zone
+		(net "Net-(F1-Pad1)")
+		(layer "F.Cu")
+		(hatch none 0.1)
+		(priority 30000)
+		(attr
+			(teardrop
+				(type padvia)
+			)
+		)
+		(connect_pads yes
+			(clearance 0)
+		)
+		(min_thickness 0.0254)
+		(fill yes
+			(island_removal_mode 1)
+		)
+		(polygon
+			(pts
+				(xy 102.0941 55.84) (xy 101.932316 55.848491) (xy 101.664992 55.86109) (xy 101.525065 55.855578)
+				(xy 101.392006 55.83486) (xy 101.274096 55.793441) (xy 101.223412 55.763251) (xy 101.17962 55.725823)
+				(xy 101.143758 55.680471) (xy 101.116861 55.626508) (xy 101.099963 55.563247) (xy 101.0941 55.49)
+				(xy 100.039 56.49) (xy 101.0941 57.49) (xy 101.09897 57.422912) (xy 101.113059 57.364149) (xy 101.134965 57.314304)
+				(xy 101.164191 57.271419) (xy 101.245451 57.202296) (xy 101.362596 57.152818) (xy 101.526271 57.124316)
+				(xy 101.749542 57.120641) (xy 101.932316 57.131509) (xy 102.0941 57.14)
+			)
+		)
+	)
+	(zone
 		(net "Net-(IC1-SEL1)")
 		(layer "F.Cu")
@@
 	)
 	(zone
-		(net "Net-(A1-D9)")
-		(layer "F.Cu")
-		(hatch none 0.1)
-		(priority 30072)
-		(attr
-			(teardrop
-				(type padvia)
-			)
-		)
-		(connect_pads yes
-			(clearance 0)
-		)
-		(min_thickness 0.0254)
-		(fill yes
-			(island_removal_mode 1)
-		)
-		(polygon
-			(pts
-				(xy 228.824893 71.199592) (xy 228.681089 71.194703) (xy 228.559584 71.180483) (xy 228.463436 71.159509)
-				(xy 228.380237 71.131602) (xy 228.238221 71.055517) (xy 228.067787 70.919674) (xy 227.877522 70.765067)
-				(xy 227.755096 70.68104) (xy 227.605862 70.594055) (xy 227.223893 71.299592) (xy 227.605862 72.005129)
-				(xy 227.841508 71.860162) (xy 228.067787 71.67951) (xy 228.206647 71.565952) (xy 228.278201 71.518212)
-				(xy 228.356759 71.477488) (xy 228.446516 71.444522) (xy 228.551662 71.420056) (xy 228.67639 71.404832)
-				(xy 228.824893 71.399592)
-			)
-		)
-	)
-	(zone
 		(net "+5V")
 		(layer "F.Cu")
@@
 	)
 	(zone
+		(net "Net-(A1-D9)")
+		(layer "F.Cu")
+		(hatch none 0.1)
+		(priority 30001)
+		(attr
+			(teardrop
+				(type padvia)
+			)
+		)
+		(connect_pads yes
+			(clearance 0)
+		)
+		(min_thickness 0.0254)
+		(fill yes
+			(island_removal_mode 1)
+		)
+		(polygon
+			(pts
+				(xy 231.117822 71.399592) (xy 231.314964 71.404241) (xy 231.475267 71.416781) (xy 231.741074 71.460549)
+				(xy 231.805783 71.474592) (xy 232.084121 71.526154) (xy 232.264317 71.543147) (xy 232.493745 71.549592)
+				(xy 232.718822 71.299592) (xy 231.752125 71.049592) (xy 231.769859 71.106418) (xy 231.772776 71.151204)
+				(xy 231.764905 71.180123) (xy 231.748516 71.202306) (xy 231.692183 71.229554) (xy 231.583549 71.237597)
+				(xy 231.385458 71.22021) (xy 231.117822 71.199592)
+			)
+		)
+	)
+	(zone
 		(net "Net-(J5-Pin_2)")
 		(layer "F.Cu")
@@
 	)
 	(zone
-		(net "Net-(F1-Pad1)")
-		(layer "F.Cu")
-		(hatch none 0.1)
-		(priority 30001)
-		(attr
-			(teardrop
-				(type padvia)
-			)
-		)
-		(connect_pads yes
-			(clearance 0)
-		)
-		(min_thickness 0.0254)
-		(fill yes
-			(island_removal_mode 1)
-		)
-		(polygon
-			(pts
-				(xy 102.0941 55.84) (xy 101.932316 55.848491) (xy 101.664992 55.86109) (xy 101.525065 55.855578)
-				(xy 101.392006 55.83486) (xy 101.274096 55.793441) (xy 101.223412 55.763251) (xy 101.17962 55.725823)
-				(xy 101.143758 55.680471) (xy 101.116861 55.626508) (xy 101.099963 55.563247) (xy 101.0941 55.49)
-				(xy 100.039 56.49) (xy 101.0941 57.49) (xy 101.09897 57.422912) (xy 101.113059 57.364149) (xy 101.134965 57.314304)
-				(xy 101.164191 57.271419) (xy 101.245451 57.202296) (xy 101.362596 57.152818) (xy 101.526271 57.124316)
-				(xy 101.749542 57.120641) (xy 101.932316 57.131509) (xy 102.0941 57.14)
-			)
-		)
-	)
-	(zone
 		(net "Net-(A1-MOSI)")
 		(layer "F.Cu")
@@
 	)
 	(zone
+		(net "Net-(IC1-S1B)")
+		(layer "F.Cu")
+		(hatch none 0.1)
+		(priority 30000)
+		(attr
+			(teardrop
+				(type padvia)
+			)
+		)
+		(connect_pads yes
+			(clearance 0)
+		)
+		(min_thickness 0.0254)
+		(fill yes
+			(island_removal_mode 1)
+		)
+		(polygon
+			(pts
+				(xy 190.051312 87.759592) (xy 190.147998 87.76441) (xy 190.220115 87.778135) (xy 190.321493 87.823522)
+				(xy 190.352674 87.842383) (xy 190.428517 87.886753) (xy 190.53394 87.936756) (xy 190.652312 87.659592)
+				(xy 190.53394 87.382428) (xy 190.376151 87.462503) (xy 190.352673 87.476801) (xy 190.294609 87.510773)
+				(xy 190.233781 87.536895) (xy 190.157059 87.553668) (xy 190.051312 87.559592)
+			)
+		)
+	)
+	(zone
 		(net "Net-(F1-Pad1)")
 		(layer "F.Cu")
 		(hatch none 0.1)
-		(priority 30003)
+		(priority 30001)
 		(attr
 			(teardrop
@@
 		(layer "F.Cu")
 		(hatch none 0.1)
-		(priority 30098)
+		(priority 30001)
 		(attr
 			(teardrop
@@
 		(layer "B.Cu")
 		(hatch none 0.1)
-		(priority 30035)
+		(priority 30000)
 		(attr
 			(teardrop

Commit message: changed molex connector
Parts:
- removed J0: 43045-0412, 43045-0412:MOLEX_43045-0412
- added J9: Conn_01x02_Pin, Connector_Molex:Molex_Micro-Fit_3.0_43650-0215_1x02_P3.00mm_Vertical, F.Cu at (114.2, 56.5)
- J1, J2, J3, J4: footprint molex_0436500215:Molex_Micro-Fit_3.0_43650-0215_1x02_P3.00mm_Vertical -> Connector_Molex:Molex_Micro-Fit_3.0_43650-0215_1x02_P3.00mm_Vertical
- moved TP2 1.68 mm to (126.5, 56.5)
Routing:
- net Net-(J9-Pin_1): track 17.9 -> 14.2 mm
- net GND: track 20.2 -> 19.7 mm
