File: hardware/control/control.kicad_pcb (KiCad board)
At the start: 2 copper layers, 200 x 70 mm, 46 parts, among them IC1 TMUX4053DYYR, J1 Conn_01x02_Pin, J11 Conn_01x04_Pin, J12 Camera Isolated triggers (ope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, J2 Conn_01x02_Pin, J3 Conn_01x02_Pin, J4 Conn_01x02_Pin, J5 Conn_01x05_Pin, J6 Conn_01x04_Pin, J7 Conn_01x08_Pin, J8 Camera Isolated triggers (ope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, J9 Conn_01x02_Pin, U2 MCP4728, U4 R-78HB12-0.5, U5 R-78HB5.0-0.5

Commit message: added schottky diode to 12V
Parts:
- added D1: 1N5817, Diode_THT:D_DO-41_SOD81_P10.16mm_Horizontal, F.Cu at (198.1, 61.0)
Connections:
- A1 pad 30: +12V -> Net-(A1-VIN)
- J6 pad 2: +12V -> Net-(A1-VIN)
Routing:
- net +12V: track 153.3 -> 13.9 mm
- net Net-(A1-VIN): track 0.00 -> 129.2 mm

Commit message: updated connectors and connector position
Parts:
- added H5: MountingHole, MountingHole:MountingHole_3.2mm_M3, F.Cu at (152.5, 55.0)
- added H6: MountingHole, MountingHole:MountingHole_3.2mm_M3, F.Cu at (152.5, 115.0)
- J1, J2, J3, J4: footprint Connector_Molex:Molex_Micro-Fit_3.0_43650-0215_1x02_P3.00mm_Vertical -> Connector_Molex:Molex_Micro-Fit_3.0_43650-0200_1x02_P3.00mm_Horizontal
- J9: value Conn_01x02_Pin -> Screw_Terminal_01x02; footprint Connector_Molex:Molex_Micro-Fit_3.0_43650-0215_1x02_P3.00mm_Vertical -> TerminalBlock_Phoenix:TerminalBlock_Phoenix_MKDS-1,5-2-5.08_1x02_P5.08mm_Horizontal
- moved TP2 87.4 mm to (60.0, 113.2)
- moved J9 74.9 mm to (52.5, 98.9), turned to -90 degrees
- moved F1 57.3 mm to (52.5, 88.4), turned to 90 degrees
- moved J4 20.3 mm to (97.8, 112.9)
- moved J1 19.8 mm to (137.2, 112.9)
- moved H1 15.0 mm to (50.0, 55.0)
- moved H4 15.0 mm to (50.0, 115.0)
- moved J3 7.03 mm to (110.9, 112.9)
- moved J2 6.54 mm to (124.1, 112.9)
Routing:
- net +48V: track 189.1 -> 212.3 mm
- net Net-(J4-Pin_2): track 20.0 -> 34.3 mm
- net Net-(J1-Pin_1): track 20.2 -> 34.4 mm
- net Net-(J1-Pin_2): track 20.0 -> 24.8 mm
- net Net-(J4-Pin_1): track 20.2 -> 24.5 mm
- net Net-(J9-Pin_1): track 14.2 -> 10.5 mm
- net GND: track 19.7 -> 22.8 mm
- net Net-(J3-Pin_1): track 20.2 -> 17.8 mm
- net Net-(J2-Pin_2): track 20.0 -> 17.9 mm
- net Net-(J3-Pin_2): track 20.0 -> 21.6 mm
- net Net-(J2-Pin_1): track 20.2 -> 21.6 mm
Other:
- board size 200 x 70 mm -> 215 x 70 mm
